File: 36C3_Badge_Hardware/36C3_Badge_Hardware.sch (KiCad schematic (older format))
At the start: 155 parts, among them J1 MicroUSB, J2 ISP, Q1 FS8205A, Q10 MMBTA42, Q2 MMBTA42, Q3 MMBTA42, Q4 MMBTA92, Q5 MMBTA42, Q6 MMBTA42, Q7 MMBTA42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

Commit message: Changed VFD footprint to have no silkscreen
Parts:
- VFD1: footprint custom:VFD_HCS-12SS59T -> custom:VFD_HCS-12SS59T_noSilk
Changed lines of the file:
@@
 F 0 "VFD1" H 14503 6890 50  0000 L CNN
 F 1 "HCS-12SS59T" H 14503 6799 50  0000 L CNN
-F 2 "custom:VFD_HCS-12SS59T" H 14850 8100 50  0001 C CNN
+F 2 "custom:VFD_HCS-12SS59T_noSilk" H 14850 8100 50  0001 C CNN
 F 3 "" H 14850 8100 50  0001 C CNN
 	1    13700 6650

Commit message: First revision of PCB
Changed lines of the file:
@@
 Sheet 1 1
 Title "36C3 Badge"
-Date "2019-12-06"
+Date "2019-12-08"
 Rev "1.0"
 Comp ""
 Comment1 "Julian Metzler"
 Comment2 "@Mezgrman"
-Comment3 ""
+Comment3 "Cato"
 Comment4 ""
 $EndDescr
@@
 L custom:VCC #PWR025
 U 1 1 5DEDF1FF
-P 5800 3400
-F 0 "#PWR025" H 5800 3250 50  0001 C CNN
-F 1 "VCC" H 5815 3573 50  0000 C CNN
-F 2 "" H 5800 3400 50  0001 C CNN
-F 3 "" H 5800 3400 50  0001 C CNN
-	1    5800 3400
+P 4350 3400
+F 0 "#PWR025" H 4350 3250 50  0001 C CNN
+F 1 "VCC" H 4365 3573 50  0000 C CNN
+F 2 "" H 4350 3400 50  0001 C CNN
+F 3 "" H 4350 3400 50  0001 C CNN
+	1    4350 3400
 	1    0    0    -1
 $EndComp
@@
 	16450 2400 16550 2400
 Wire Wire Line
-	4350 3650 4350 3900
-Wire Wire Line
 	4200 4900 5150 4900
 Connection ~ 4950 4700
@@
 $EndComp
 Connection ~ 3750 2350
-$Comp
-L power:PWR_FLAG #FLG0106
-U 1 1 5EB4BC05
-P 5800 3850
-F 0 "#FLG0106" H 5800 3925 50  0001 C CNN
-F 1 "PWR_FLAG" V 5800 3978 50  0000 L CNN
-F 2 "" H 5800 3850 50  0001 C CNN
-F 3 "~" H 5800 3850 50  0001 C CNN
-	1    5800 3850
-	0    -1   -1   0
-$EndComp
 Wire Wire Line
 	4400 2100 4400 2200
@@
 	3000 6500 3000 6600
 Connection ~ 3000 6600
-Wire Wire Line
-	5800 3400 5800 3650
-Wire Wire Line
-	4350 3650 5800 3650
-Connection ~ 5800 3650
-Wire Wire Line
-	5800 3650 5800 3850
 $Comp
 L custom:VCC #PWR0102
@@
 	1    0    0    -1
 $EndComp
+Wire Wire Line
+	4350 3400 4350 3900
 $EndSCHEMATC

Commit message: Schematic / Board updates and bugfixes:
- Updated crack LED resistor values after testing
- Changed microcontroller reset capacitor from 100nF to 1µF and case from 0603 to 0805
- Changed MMBTA type transistors to BC types (MMBTA didn't work in the VFD filament H-Bridge)
- Added Schottky diode in series to CH330 VCC pin. This fixes an error where the badge would erroneously detect USB power when the CH330 was backfed via the high Tx pin.
Parts:
- removed D59: 1N4148, Diodes_SMD:D_0603, symbol device:D
- added D6: BAT46W, Diodes_SMD:D_SOD-123, symbol diode:BAT46
- C27: value 100n -> 1µ; footprint Capacitors_SMD:C_0603 -> Capacitors_SMD:C_0805
- Q10, Q2, Q3, Q5, Q6, Q7, Q9: value MMBTA42 -> BC817
- Q4, Q8: value MMBTA92 -> BC807
- R14, R15, R17, R18, R19, R23, R24: value 1k -> 470R
- R26, R27, R28, R29, R33, R34: value 1k -> 2.2k
Connections:
- net +5V_USB: now also D6.2 (A); no longer C4.2, U4.5 (VCC)
- net at JP1.1 (A): now also D58.1 (K)
- new net: C4.2, D6.1 (K), U4.5 (VCC)
Other:
- moved on the sheet: D57, D58
